File: ams1117_power.kicad_sch (KiCad schematic)
At the start: 10 parts

Commit message: new pre-fabrication
Parts:
- C17: value 10 uF -> 10uF
Changed lines of the file:
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@@
       (effects (font (size 1.27 1.27)) (justify left))
     )
-    (property "Value" "10 uF" (id 1) (at 175.26 93.0909 0)
+    (property "Value" "10uF" (id 1) (at 175.26 93.0909 0)
       (effects (font (size 1.27 1.27)) (justify left))
     )
