File: esp32_4_relay.kicad_sch (KiCad schematic)
At the start: 26 parts

Commit message: pre-production
Parts:
- ESP32S3: LCSC (none) -> C2913204
Connections:
- net IO21: now also LEDU1.1 (K)
- net IO45: no longer LEDU1.1 (K)
Other:
- moved on the sheet: LEDU1, RLEDUV1

Commit message: new pre-fabrication
Parts:
- C1, C2, C3, C4: value 100 nF -> 100nF
- CONNL1, CONNPOW1, CONNR1, DRA1, DRA2, ESP323V3, H1, H2: now left out of the parts list
- F1: LCSC (none) -> C84140
