File: relay_1.kicad_sch (KiCad schematic)
At the start: 44 parts, among them Q1 L8050QLT1G, Q2 L8050QLT1G, Q3 L8050QLT1G, Q4 L8050QLT1G, SW1 SW_Push_DPDT, SW2 SW_Push_DPDT, SW3 SW_Push_DPDT, SW4 SW_Push_DPDT, U1 PC817, U2 PC817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

Commit message: pre-production
Parts:
- DRR1, DRR2, DRR3, DRR4: footprint LED_SMD:LED_1206_3216Metric -> LED_SMD:LED_0805_2012Metric
Other:
- moved on the sheet: JR1, JR3

Commit message: new pre-fabrication
Parts:
- RRQOPT1, RRQOPT2, RRQOPT3, RRQOPT4: now in the parts list
Changed lines of the file:
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@@
   )
   (symbol (lib_id "Device:R") (at 204.47 67.31 0) (unit 1)
-    (in_bom no) (on_board yes)
+    (in_bom yes) (on_board yes)
     (property "Reference" "RRQOPT3" (id 0) (at 201.93 66.04 0)
       (effects (font (size 1.27 1.27)) (justify right))
@@
   )
   (symbol (lib_id "Device:R") (at 69.85 66.04 0) (unit 1)
-    (in_bom no) (on_board yes)
+    (in_bom yes) (on_board yes)
     (property "Reference" "RRQOPT1" (id 0) (at 67.31 64.77 0)
       (effects (font (size 1.27 1.27)) (justify right))
@@
   )
   (symbol (lib_id "Device:R") (at 78.74 134.62 0) (unit 1)
-    (in_bom no) (on_board yes)
+    (in_bom yes) (on_board yes)
     (property "Reference" "RRQOPT2" (id 0) (at 76.2 133.35 0)
       (effects (font (size 1.27 1.27)) (justify right))
@@
   )
   (symbol (lib_id "Device:R") (at 207.01 134.62 0) (unit 1)
-    (in_bom no) (on_board yes)
+    (in_bom yes) (on_board yes)
     (property "Reference" "RRQOPT4" (id 0) (at 204.47 133.35 0)
       (effects (font (size 1.27 1.27)) (justify right))
