File: sensors.kicad_sch (KiCad schematic)
At the start: 10 parts, among them U5 TMP75AIDR

Commit message: new pre-fabrication
Parts:
- removed CTMP1: 100 nF, Capacitor_SMD:C_0805_2012Metric, symbol Device:C
- removed RTMP1: 4K7, Resistor_SMD:R_0805_2012Metric, symbol Device:R
- removed U5: TMP75AIDR, Package_SO:SOIC-8_3.9x4.9mm_P1.27mm, symbol TMP75AIDR:TMP75AIDR
- added C18: 100nF, Capacitor_SMD:C_0805_2012Metric, symbol Device:C
- added U5: HDC1080, Package_SON:Texas_PWSON-N6, symbol Sensor_Humidity:HDC1080
- I2C1, I2C2: now left out of the parts list
Connections:
- net +3.3V: now also C18.1, U5.5 (VCC)
- net GND: now also C18.2, U5.2 (GND)
- net S_SCL: now also U5.6 (SCL)
- net S_SDA: now also U5.1 (SDA)
Other:
- note added: "The I2C address of the HDC1080 is 1000000 (7-bit address"
- note added: "https://www.ti.com/lit/ds/symlink/hdc1080.pdf"
- note removed: "ADDR to GND, so addr will be 1001000"
- note removed: "TMP75 sensor"
- note removed: "https://www.ti.com/lit/ds/symlink/tmp75.pdf"
- note removed: "we dont need alert"
