File: esp32_4_relay.kicad_pcb (KiCad board)
At the start: 4 copper layers, 124 x 95 mm, 122 parts, among them Q1 L8050QLT1G, Q2 L8050QLT1G, Q3 L8050QLT1G, Q4 L8050QLT1G, Q5 L8050QLT1G, Q6 L8050QLT1G, Q7 2N7002, SW1 SW_Push_DPDT, SW2 SW_Push_DPDT, SW3 SW_Push_DPDT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

Commit message: pre-production
Parts:
- DRR1, DRR2, DRR3, DRR4: footprint LED_SMD:LED_1206_3216Metric -> LED_SMD:LED_0805_2012Metric
- R10, R12: value 1M -> 5.1K
- moved RDS1 25.6 mm to (205.2, 110.0), turned to 180 degrees
- moved R3 16.5 mm to (105.2, 64.5), turned to 90 degrees
- moved R12 15.3 mm to (116.5, 72.5)
- moved 3V1 15.1 mm to (123.3, 76.8)
- moved C15 13.9 mm to (127.6, 90.7), turned to 0 degrees
- moved C16 11.8 mm to (121.5, 90.5), turned to 180 degrees
- moved C9 9.91 mm to (105.1, 76.5), turned to 90 degrees
- moved RTMP1 9.60 mm to (192.6, 104.5), turned to -90 degrees
- moved R2 8.86 mm to (216.1, 72.5), turned to -90 degrees
- moved D7 8.54 mm to (114.0, 70.5), turned to 0 degrees
- moved RI2C2 7.20 mm to (202.4, 97.1), turned to 0 degrees
- moved C5 7.18 mm to (180.1, 89.2), turned to 180 degrees
- moved R11 7.09 mm to (180.0, 84.5)
- moved RI2C1 7.07 mm to (197.5, 97.0), turned to 180 degrees
- moved D5 6.71 mm to (110.5, 70.5), turned to 180 degrees
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Connections:
- DS1 pad 2: /IO21 -> /IO45
- DS2 pad 2: /IO21 -> /IO45
- LEDU1 pad 1: /IO45 -> /IO21
- RDS1 pad 2: /IO21 -> /IO45
- ROPT1 pad 1: /IO10 -> /IO13
- ROPT2 pad 1: /IO11 -> /IO12
- ROPT3 pad 1: /IO12 -> /IO11
- ROPT4 pad 1: /IO13 -> /IO10
Routing:
- net /5V_WORK: track 20.2 -> 247.5 mm
- net /USBC_CP2102/VBUS: track 0.00 -> 76.5 mm
- net /IO10: track 83.1 -> 152.7 mm, vias 1 -> 2
- net GND: track 54.7 -> 124.3 mm, vias 17 -> 101
- net /IO45: track 86.5 -> 147.3 mm
- net +3.3V: track 26.1 -> 80.9 mm, vias 4 -> 19
- net /IO11: track 88.7 -> 140.7 mm, vias 1 -> 2
- net Net-(D1-Pad2): track 0.00 -> 41.9 mm
- net Net-(D2-Pad2): track 0.00 -> 40.4 mm
- net Net-(D3-Pad2): track 0.00 -> 39.1 mm
- net /CP2102_RX: track 0.00 -> 38.8 mm
- net /USBC_CP2102/USB_N: track 15.9 -> 53.5 mm
- net /IO48: track 98.4 -> 134.9 mm
- net /USBC_CP2102/USB_P: track 17.0 -> 53.2 mm, vias 0 -> 2
- net /CP2102_TX: track 0.00 -> 35.6 mm
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- added copper zone on B.Cu, net GND
Other:
- board text added: "3V3"
- board text added: "3V3TP"
- board text added: "3V3TP ESPIN"
- board text added: "45/DS"
- board text added: "47/SCL"
- board text added: "48/SDA"
- board text added: "5V"
- board text added: "5V FROM PINS OR SCREWS"
- board text added: "5V FROM USB"
- board text added: "5V INPUT"
- board text added: "5VTP"
- board text added: "5V_IN"
- board text added: "AMS1117"
- board text added: "COMM"
- board text added: "CP2101N"
- board text added: "DATA"
- board text added: "DS18B20 CONNECTION"
- board text added: "EN"
- board text added: "GND"
- board text added: "I2C PINS"
- board text added: "IO0"
- board text added: "IO1"
- board text added: "IO10/REL4"
- board text added: "IO11/REL3"
- board text added: "IO12/REL2"
- board text added: "IO13/REL1"
- board text added: "IO14"
- board text added: "IO15"
- board text added: "IO16"
- board text added: "IO17"
- board text added: "IO18"
- board text added: "IO19"
- board text added: "IO2"
- board text added: "IO20"
- board text added: "IO21/L"
- board text added: "IO3"
- board text added: "IO38"
- board text added: "IO39"
- board text added: "IO4"
- board text added: "IO40"
- board text added: "IO41"
- board text added: "IO42"
- board text added: "IO46"
- board text added: "IO5"
- board text added: "IO6"
- board text added: "IO7"
- board text added: "IO8"
- board text added: "IO9"
- board text added: "NC"
- board text added: "NO"
- board text added: "RELAY1"
- board text added: "RELAY2"
- board text added: "RELAY3"
- board text added: "RELAY4"
- board text added: "REMOVE R9 TO SET DIFF POWER FOR ESP"
- board text added: "RX0"
- board text added: "SCL"
- board text added: "SDA"
- board text added: "TX0"
- board text added: "VBUSTP"
- board text added: "Согласно таблицам расстояний путей утечки, расстояние от дорожки 220В до другой в 3 мм вполне безопасно, так что воздушных зазоров не делаем, это будет очень дорого"

Commit message: new pre-fabrication
Parts:
- removed CTMP1: 100 nF, Capacitor_SMD:C_0805_2012Metric
- removed RTMP1: 4K7, Resistor_SMD:R_0805_2012Metric
- removed SW5, SW6: SW_DIP_x01, Button_Switch_SMD:SW_Push_1P1T_NO_6x6mm_H9.5mm
- added C18: 100nF, Capacitor_SMD:C_0805_2012Metric, F.Cu at (199.2, 100.5)
- added S1: TS-1187A-B-A-B, TS-1187A-B-A-B:SW_TS-1187A-B-A-B, F.Cu at (173.1, 86.2)
- added S2: TS-1187A-B-A-B, TS-1187A-B-A-B:SW_TS-1187A-B-A-B, F.Cu at (188.4, 86.3)
- C1, C2, C3, C4: value 100 nF -> 100nF
- C17: value 10 uF -> 10uF
- R10, R12: value 5.1K -> 5K1
- U5: value TMP75AIDR -> HDC1080; footprint Package_SO:SOIC-8_3.9x4.9mm_P1.27mm -> Package_SON:Texas_PWSON-N6
- moved I2C2 9.68 mm to (194.5, 108.3), turned to 0 degrees
- moved I2C1 7.76 mm to (198.5, 108.3), turned to 0 degrees
- moved U5 1.30 mm to (199.2, 103.5), turned to 180 degrees
Connections:
- U5 pad 2: /IO47 -> GND
- U5 pad 3: Net-(RTMP1-Pad1) -> unconnected-(U5-Pad3)
- U5 pad 4: GND -> unconnected-(U5-Pad4)
- U5 pad 5: GND -> +3.3V
- U5 pad 6: GND -> /IO47
- U5 pad 7: GND -> unconnected-(U5-Pad7)
Routing:
- net Net-(R3-Pad1): track 20.1 -> 3.13 mm
- net GND: track 124.3 -> 128.7 mm, vias 101 -> 129
- net Net-(RTMP1-Pad1): track 3.34 -> 0.00 mm
- net /IO48: track 134.9 -> 132.0 mm
- net /IO47: track 140.6 -> 142.1 mm
- net +3.3V: track 80.9 -> 82.3 mm, vias 19 -> 18
- net Net-(C5-Pad2): track 14.9 -> 13.9 mm
- net Net-(C10-Pad2): track 14.6 -> 14.1 mm
- net /5V_PINS: track 107.6 -> 107.0 mm
Other:
- board text added: "BOOT"
- board text added: "RESET"

Commit message: production
Parts:
- added G***: LOGO, LOGO, F.Cu at (186.3, 73.2)
- moved R8 3.38 mm to (180.2, 81.0)
- moved R7 2.43 mm to (177.6, 81.0)
- moved C14 0.35 mm to (132.7, 87.4)
- moved C17 0.25 mm to (114.0, 82.6)
Routing:
- net /5V_WORK: track 247.5 -> 241.5 mm
- net /TX0: track 88.2 -> 92.9 mm
- net /RX0: track 91.0 -> 95.3 mm
- net /CP2102_RX: track 38.8 -> 36.0 mm
- net /CP2102_TX: track 35.6 -> 33.1 mm
- net /EN: track 92.9 -> 91.9 mm
- net GND: vias 129 -> 128
Other:
- board text added: "HOW TO USE 3-PIN POWER SELECTOR: The jumper allows you to change the 5V supply source from the pins or from the USB. By removing the jumper, you can apply 3.3V directly from an external source. Then the relays will be de-energized. If you connect all three pins, then 5V from the USB will be available on the pins and screw connector."
- board text added: "KOLOS v2.0, 2023"
- board text added: "Power selector"
