File: usbc_cp2102.kicad_sch (KiCad schematic)
At the start: 32 parts, among them Q5 L8050QLT1G, Q6 L8050QLT1G, Q7 2N7002, SW5 SW_DIP_x01, SW6 SW_DIP_x01

Commit message: pre-production
Parts:
- R10, R12: value 1M -> 5.1K
Changed lines of the file:
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@@
       (effects (font (size 1.27 1.27)) (justify left))
     )
-    (property "Value" "1M" (id 1) (at 92.71 69.8499 0)
+    (property "Value" "5.1K" (id 1) (at 92.71 69.8499 0)
       (effects (font (size 1.27 1.27)) (justify left))
     )
@@
       (effects (font (size 1.27 1.27)) (justify left))
     )
-    (property "Value" "1M" (id 1) (at 85.09 69.8499 0)
-      (effects (font (size 1.27 1.27)) (justify left))
-    )
+    (property "Value" "5.1K" (id 1) (at 85.09 69.8499 0)
+      (effects (font (size 1.27 1.27)) (justify left))
+    )

Commit message: new pre-fabrication
Parts:
- removed SW5, SW6: SW_DIP_x01, Button_Switch_SMD:SW_Push_1P1T_NO_6x6mm_H9.5mm, symbol Switch:SW_DIP_x01
- added S1, S2: TS-1187A-B-A-B, TS-1187A-B-A-B:SW_TS-1187A-B-A-B, symbol TS-1187A-B-A-B:TS-1187A-B-A-B
- 5V1, C10, C5, R19, VBUS1: now left out of the parts list
- R10, R12: value 5.1K -> 5K1
Connections:
- net GND: now also S1.A, S1.B, S2.A, S2.B
- net at C5.2, R11.1: now also S1.C, S1.D
- net at C10.2, R15.1: now also S2.C, S2.D
Changed lines of the file:
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@@
     (pin "3")
+  )
+  (symbol (lib_id "TS-1187A-B-A-B:TS-1187A-B-A-B") (at 66.04 137.16 0) (unit 1)
+    (in_bom yes) (on_board yes) (fields_autoplaced)
+    (property "Reference" "S1" (id 0) (at 66.04 129.54 0))
+    (property "Value" "TS-1187A-B-A-B" (id 1) (at 66.04 132.08 0))
+    (property "Footprint" "TS-1187A-B-A-B:SW_TS-1187A-B-A-B" (id 2) (at 66.04 137.16 0)
+      (effects (font (size 1.27 1.27)) (justify bottom) hide)
+    )
+    (property "Datasheet" "" (id 3) (at 66.04 137.16 0)
+      (effects (font (size 1.27 1.27)) hide)
+    )
+    (property "PARTREV" "A0" (id 4) (at 66.04 137.16 0)
+      (effects (font (size 1.27 1.27)) (justify bottom) hide)
+    )
+    (property "MANUFACTURER" "XKB Industrial Precision" (id 5) (at 66.04 137.16 0)
+      (effects (font (size 1.27 1.27)) (justify bottom) hide)
+    )
+    (property "MAXIMUM_PACKAGE_HEIGHT" "1.5mm" (id 6) (at 66.04 137.16 0)
+      (effects (font (size 1.27 1.27)) (justify bottom) hide)
+    )
+    (property "STANDARD" "Manufacturer Recommendations" (id 7) (at 66.04 137.16 0)
+      (effects (font (size 1.27 1.27)) (justify bottom) hide)
+    )
+    (pin "A")
+    (pin "B")
+    (pin "C")
+    (pin "D")
   )
   (symbol (lib_id "Device:R") (at 66.04 180.34 270) (unit 1)
@@
     (pin "1")
   )
+  (symbol (lib_id "TS-1187A-B-A-B:TS-1187A-B-A-B") (at 107.95 137.16 0) (unit 1)
+    (in_bom yes) (on_board yes) (fields_autoplaced)
+    (property "Reference" "S2" (id 0) (at 107.95 129.54 0))
+    (property "Value" "TS-1187A-B-A-B" (id 1) (at 107.95 132.08 0))
+    (property "Footprint" "TS-1187A-B-A-B:SW_TS-1187A-B-A-B" (id 2) (at 107.95 137.16 0)
+      (effects (font (size 1.27 1.27)) (justify bottom) hide)
+    )
+    (property "Datasheet" "" (id 3) (at 107.95 137.16 0)
+      (effects (font (size 1.27 1.27)) hide)
+    )
+    (property "PARTREV" "A0" (id 4) (at 107.95 137.16 0)
+      (effects (font (size 1.27 1.27)) (justify bottom) hide)
+    )
+    (property "MANUFACTURER" "XKB Industrial Precision" (id 5) (at 107.95 137.16 0)
+      (effects (font (size 1.27 1.27)) (justify bottom) hide)
+    )
+    (property "MAXIMUM_PACKAGE_HEIGHT" "1.5mm" (id 6) (at 107.95 137.16 0)
+      (effects (font (size 1.27 1.27)) (justify bottom) hide)
+    )
+    (property "STANDARD" "Manufacturer Recommendations" (id 7) (at 107.95 137.16 0)
+      (effects (font (size 1.27 1.27)) (justify bottom) hide)
+    )
+    (pin "A")
+    (pin "B")
+    (pin "C")
+    (pin "D")
+  )
   (symbol (lib_id "power:GND") (at 176.53 91.44 0) (unit 1)
     (in_bom yes) (on_board yes) (fields_autoplaced)
@@
       (effects (font (size 1.27 1.27)) (justify left))
     )
-    (property "Value" "5.1K" (id 1) (at 92.71 69.8499 0)
+    (property "Value" "5K1" (id 1) (at 92.71 69.8499 0)
       (effects (font (size 1.27 1.27)) (justify left))
     )
@@
   )
   (symbol (lib_id "Device:R") (at 246.38 54.61 0) (unit 1)
-    (in_bom yes) (on_board yes) (fields_autoplaced)
+    (in_bom no) (on_board yes) (fields_autoplaced)
     (property "Reference" "R19" (id 0) (at 248.92 53.3399 0)
       (effects (font (size 1.27 1.27)) (justify left))
@@
   )
   (symbol (lib_id "Connector:TestPoint") (at 72.39 46.99 0) (unit 1)
-    (in_bom yes) (on_board yes)
+    (in_bom no) (on_board yes)
     (property "Reference" "5V1" (id 0) (at 71.12 38.1 0)
       (effects (font (size 1.27 1.27)) (justify left))
@@
     (pin "2")
   )
-  (symbol (lib_id "Switch:SW_DIP_x01") (at 66.04 137.16 0) (unit 1)
-    (in_bom yes) (on_board yes) (fields_autoplaced)
-    (property "Reference" "SW5" (id 0) (at 66.04 129.54 0))
-    (property "Value" "SW_DIP_x01" (id 1) (at 66.04 132.08 0))
-    (property "Footprint" "Button_Switch_SMD:SW_Push_1P1T_NO_6x6mm_H9.5mm" (id 2) (at 66.04 137.16 0)
-      (effects (font (size 1.27 1.27)) hide)
-    )
-    (property "Datasheet" "~" (id 3) (at 66.04 137.16 0)
-      (effects (font (size 1.27 1.27)) hide)
-    )
-    (pin "1")
-    (pin "2")
-  )
   (symbol (lib_id "power:GND") (at 242.57 99.06 0) (unit 1)
     (in_bom yes) (on_board yes) (fields_autoplaced)
@@
   )
   (symbol (lib_id "Connector:TestPoint") (at 57.15 46.99 0) (unit 1)
-    (in_bom yes) (on_board yes)
+    (in_bom no) (on_board yes)
     (property "Reference" "VBUS1" (id 0) (at 55.88 38.1 0)
       (effects (font (size 1.27 1.27)) (justify left))
@@
   )
   (symbol (lib_id "Device:C") (at 68.58 143.51 90) (unit 1)
-    (in_bom yes) (on_board yes)
+    (in_bom no) (on_board yes)
     (property "Reference" "C5" (id 0) (at 68.58 147.32 90))
     (property "Value" "100 nF" (id 1) (at 68.58 149.86 90))
@@
   )
   (symbol (lib_id "Device:C") (at 109.22 143.51 90) (unit 1)
-    (in_bom yes) (on_board yes)
+    (in_bom no) (on_board yes)
     (property "Reference" "C10" (id 0) (at 109.22 147.32 90))
     (property "Value" "100 nF" (id 1) (at 109.22 149.86 90))
@@
     (pin "2")
   )
-  (symbol (lib_id "Switch:SW_DIP_x01") (at 107.95 137.16 0) (unit 1)
-    (in_bom yes) (on_board yes) (fields_autoplaced)
-    (property "Reference" "SW6" (id 0) (at 107.95 129.54 0))
-    (property "Value" "SW_DIP_x01" (id 1) (at 107.95 132.08 0))
-    (property "Footprint" "Button_Switch_SMD:SW_Push_1P1T_NO_6x6mm_H9.5mm" (id 2) (at 107.95 137.16 0)
-      (effects (font (size 1.27 1.27)) hide)
-    )
-    (property "Datasheet" "~" (id 3) (at 107.95 137.16 0)
-      (effects (font (size 1.27 1.27)) hide)
-    )
-    (pin "1")
-    (pin "2")
-  )
   (symbol (lib_id "LESD5D5.0CT1G:LESD5D5.0CT1G") (at 68.58 82.55 270) (unit 1)
     (in_bom yes) (on_board yes) (fields_autoplaced)
@@
       (effects (font (size 1.27 1.27)) (justify left))
     )
-    (property "Value" "5.1K" (id 1) (at 85.09 69.8499 0)
-      (effects (font (size 1.27 1.27)) (justify left))
-    )
+    (property "Value" "5K1" (id 1) (at 85.09 69.8499 0)
+      (effects (font (size 1.27 1.27)) (justify left))
+    )

Commit message: fix cp2102 transistor
Parts:
- Q7: now left out of the parts list
Other:
- note added: "DO not connect this transistor until it is really need"
Changed lines of the file:
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@@
+    (effects (font (size 1.27 1.27)) (justify left bottom))
+  )
+  (text "DO not connect \nthis transistor\nuntil it is really need"
+    (at 165.1 91.44 0)
     (effects (font (size 1.27 1.27)) (justify left bottom))
   )
@@
   (text "NC" (at 69.85 146.05 0)
     (effects (font (size 1.27 1.27) (thickness 0.254) bold) (justify left bottom))
+  )
+  (text "NC" (at 172.72 85.09 0)
+    (effects (font (size 1.27 1.27)) (justify left bottom))
   )
   (text "NC" (at 110.49 146.05 0)
@@
   )
   (symbol (lib_id "Transistor_FET:2N7002") (at 179.07 80.01 0) (mirror y) (unit 1)
-    (in_bom yes) (on_board yes) (fields_autoplaced)
+    (in_bom no) (on_board yes) (fields_autoplaced)
     (property "Reference" "Q7" (id 0) (at 172.72 78.7399 0)
       (effects (font (size 1.27 1.27)) (justify left))
